Commit message: gripper_update

File: ur_simulation_gz/urdf/robotiq_gripper_macro.xacro (robot description, xacro)
@@ -43,10 +43,10 @@
             <visual>
                 <geometry>
-                    <mesh filename="package://robotiq_description/meshes/visual/2f_85/robotiq_base.dae" />
-                </geometry>
-            </visual>
-            <collision>
-                <geometry>
-                    <mesh filename="package://robotiq_description/meshes/collision/2f_85/robotiq_base.stl" />
+                    <mesh filename="package://ur_simulation_gz/meshes/visual/2f_85/robotiq_base.dae" />
+                </geometry>
+            </visual>
+            <collision>
+                <geometry>
+                    <mesh filename="package://ur_simulation_gz/meshes/collision/2f_85/robotiq_base.stl" />
                 </geometry>
             </collision>
@@ -60,10 +60,10 @@
             <visual>
                 <geometry>
-                    <mesh filename="package://robotiq_description/meshes/visual/2f_85/left_knuckle.dae" />
-                </geometry>
-            </visual>
-            <collision>
-                <geometry>
-                    <mesh filename="package://robotiq_description/meshes/collision/2f_85/left_knuckle.stl" />
+                    <mesh filename="package://ur_simulation_gz/meshes/visual/2f_85/left_knuckle.dae" />
+                </geometry>
+            </visual>
+            <collision>
+                <geometry>
+                    <mesh filename="package://ur_simulation_gz/meshes/collision/2f_85/left_knuckle.stl" />
                 </geometry>
             </collision>
@@ -77,10 +77,10 @@
             <visual>
                 <geometry>
-                    <mesh filename="package://robotiq_description/meshes/visual/2f_85/right_knuckle.dae" />
-                </geometry>
-            </visual>
-            <collision>
-                <geometry>
-                    <mesh filename="package://robotiq_description/meshes/collision/2f_85/right_knuckle.stl" />
+                    <mesh filename="package://ur_simulation_gz/meshes/visual/2f_85/right_knuckle.dae" />
+                </geometry>
+            </visual>
+            <collision>
+                <geometry>
+                    <mesh filename="package://ur_simulation_gz/meshes/collision/2f_85/right_knuckle.stl" />
                 </geometry>
             </collision>
@@ -94,10 +94,10 @@
             <visual>
                 <geometry>
-                    <mesh filename="package://robotiq_description/meshes/visual/2f_85/left_finger.dae" />
-                </geometry>
-            </visual>
-            <collision>
-                <geometry>
-                    <mesh filename="package://robotiq_description/meshes/collision/2f_85/left_finger.stl" />
+                    <mesh filename="package://ur_simulation_gz/meshes/visual/2f_85/left_finger.dae" />
+                </geometry>
+            </visual>
+            <collision>
+                <geometry>
+                    <mesh filename="package://ur_simulation_gz/meshes/collision/2f_85/left_finger.stl" />
                 </geometry>
             </collision>
@@ -111,10 +111,10 @@
             <visual>
                 <geometry>
-                    <mesh filename="package://robotiq_description/meshes/visual/2f_85/right_finger.dae" />
-                </geometry>
-            </visual>
-            <collision>
-                <geometry>
-                    <mesh filename="package://robotiq_description/meshes/collision/2f_85/right_finger.stl" />
+                    <mesh filename="package://ur_simulation_gz/meshes/visual/2f_85/right_finger.dae" />
+                </geometry>
+            </visual>
+            <collision>
+                <geometry>
+                    <mesh filename="package://ur_simulation_gz/meshes/collision/2f_85/right_finger.stl" />
                 </geometry>
             </collision>
@@ -128,10 +128,10 @@
             <visual>
                 <geometry>
-                    <mesh filename="package://robotiq_description/meshes/visual/2f_85/left_inner_knuckle.dae" />
-                </geometry>
-            </visual>
-            <collision>
-                <geometry>
-                    <mesh filename="package://robotiq_description/meshes/collision/2f_85/left_inner_knuckle.stl" />
+                    <mesh filename="package://ur_simulation_gz/meshes/visual/2f_85/left_inner_knuckle.dae" />
+                </geometry>
+            </visual>
+            <collision>
+                <geometry>
+                    <mesh filename="package://ur_simulation_gz/meshes/collision/2f_85/left_inner_knuckle.stl" />
                 </geometry>
             </collision>
@@ -145,10 +145,10 @@
             <visual>
                 <geometry>
-                    <mesh filename="package://robotiq_description/meshes/visual/2f_85/right_inner_knuckle.dae" />
-                </geometry>
-            </visual>
-            <collision>
-                <geometry>
-                    <mesh filename="package://robotiq_description/meshes/collision/2f_85/right_inner_knuckle.stl" />
+                    <mesh filename="package://ur_simulation_gz/meshes/visual/2f_85/right_inner_knuckle.dae" />
+                </geometry>
+            </visual>
+            <collision>
+                <geometry>
+                    <mesh filename="package://ur_simulation_gz/meshes/collision/2f_85/right_inner_knuckle.stl" />
                 </geometry>
             </collision>
@@ -162,10 +162,10 @@
             <visual>
                 <geometry>
-                    <mesh filename="package://robotiq_description/meshes/visual/2f_85/left_finger_tip.dae" />
-                </geometry>
-            </visual>
-            <collision>
-                <geometry>
-                    <mesh filename="package://robotiq_description/meshes/collision/2f_85/left_finger_tip.stl" />
+                    <mesh filename="package://ur_simulation_gz/meshes/visual/2f_85/left_finger_tip.dae" />
+                </geometry>
+            </visual>
+            <collision>
+                <geometry>
+                    <mesh filename="package://ur_simulation_gz/meshes/collision/2f_85/left_finger_tip.stl" />
                 </geometry>
                 <surface>
@@ -197,10 +197,10 @@
             <visual>
                 <geometry>
-                    <mesh filename="package://robotiq_description/meshes/visual/2f_85/right_finger_tip.dae" />
-                </geometry>
-            </visual>
-            <collision>
-                <geometry>
-                    <mesh filename="package://robotiq_description/meshes/collision/2f_85/right_finger_tip.stl" />
+                    <mesh filename="package://ur_simulation_gz/meshes/visual/2f_85/right_finger_tip.dae" />
+                </geometry>
+            </visual>
+            <collision>
+                <geometry>
+                    <mesh filename="package://ur_simulation_gz/meshes/collision/2f_85/right_finger_tip.stl" />
                 </geometry>
                 <surface>
