Commit message: add camera, table and tower to sim

File: ur_simulation_gz/urdf/ur5_gripper.urdf.xacro (robot description, xacro)
@@ -53,4 +53,9 @@
    <!-- create link fixed to the "world" -->
    <link name="world" />
+   <joint name="world_to_bot_base" type="fixed">
+    <parent link="world"/>
+    <child link="bot_base_link"/>
+    <origin xyz="0 0 0" rpy="0 0 0"/>
+  </joint>
    <xacro:if value="${is_sim_gazebo or is_sim_ignition}">
      <link name="ground_plane">
@@ -64,10 +69,10 @@
          </material>
        </visual>
-       <collision>
+       <!--<collision>
          <origin rpy="0 0 0" xyz="0 0 0"/>
          <geometry>
            <box size="5 5 0"/>
          </geometry>
-       </collision>
+       </collision>-->
      </link>
      <joint name="ground_plane_joint" type="fixed">
@@ -115,5 +120,5 @@
      trajectory_port="$(arg trajectory_port)"
      >
-     <origin xyz="0 0 0.8" rpy="0 0 0" />          <!-- position robot in the world -->
+     <origin xyz="0 0 0" rpy="0 0 0" />         <!-- position robot in the world -->
    </xacro:ur_robot>
    <xacro:if value="$(arg sim_gazebo)">
@@ -145,3 +150,149 @@
     <origin xyz="0 0 0" rpy="0 0 0" />
   </xacro:robotiq_gripper>
+  <!-- Base -->
+  <link name="bot_base_link">
+    <visual>
+      <origin xyz="0 0 0.05" rpy="0 0 0"/>
+      <geometry>
+        <cylinder length="0.1" radius="0.2"/>
+      </geometry>
+      <material name="dark_gray">
+        <color rgba="0.2 0.2 0.2 1"/>
+      </material>
+    </visual>
+    <!--<collision>
+      <origin xyz="0 0 0.05" rpy="0 0 0"/>
+      <geometry>
+        <cylinder length="0.1" radius="0.2"/>
+      </geometry>
+    </collision>-->
+  </link>
+  <joint name="robot_to_turtlebot_base" type="fixed">
+    <parent link="bot_base_link"/>
+    <child link="base_link"/>  <!-- Ur5 Base -->
+    <origin xyz="0 0 0.1" rpy="0 0 0"/>
+  </joint>
+  <!-- Tower -->
+  <link name="tower_link">
+    <visual>
+      <origin xyz="0 0 0.2" rpy="0 0 0"/>
+      <geometry>
+        <box size="0.04 0.1 1.2"/>
+      </geometry>
+      <material name="gray">
+        <color rgba="0.5 0.5 0.5 1"/>
+      </material>
+    </visual>
+    <!--<collision>
+      <origin xyz="0 0 0.2" rpy="0 0 0"/>
+      <geometry>
+        <box size="0.04 0.1 1.2"/>
+      </geometry>
+    </collision> -->
+  </link>
+  <joint name="pole_to_base" type="fixed">
+    <parent link="bot_base_link"/>
+    <child link="tower_link"/>
+    <origin xyz="-0.12 0 0.5" rpy="0 0 0"/>
+  </joint>
+  <!-- Camera -->
+  <link name="camera_link">
+    <visual>
+      <origin xyz="0 0 0" rpy="0 0 0"/>
+      <geometry>
+        <box size="0.06 0.03 0.02"/>
+      </geometry>
+      <material name="dark_gray">
+        <color rgba="0.2 0.2 0.2 1"/>
+      </material>
+    </visual>
+    <!--<collision>
+      <origin xyz="0 0 0" rpy="0 0 0"/>
+      <geometry>
+        <box size="0.06 0.03 0.02"/>
+      </geometry>
+    </collision>-->
+  </link>
+  <joint name="camera_on_pole" type="fixed">
+    <parent link="tower_link"/>
+    <child link="camera_link"/>
+    <origin xyz="0.04 0 0.7" rpy="0 0 0"/>
+  </joint>
+  <!-- Table -->
+    <link name="table_link">
+    <!-- Tischplatte -->
+    <visual>
+      <origin xyz="0 0 0.47" rpy="0 0 0"/>
+      <geometry>
+        <box size="0.67 1.0 0.033"/>
+      </geometry>
+      <material name="brown">
+        <color rgba="0.55 0.27 0.07 1"/>
+      </material>
+    </visual>
+    <collision>
+      <origin xyz="0 0 0.47" rpy="0 0 0"/>
+      <geometry>
+        <box size="0.67 1.0 0.033"/>
+      </geometry>
+    </collision>
+    <!-- Tischbeine -->
+    <visual>
+      <origin xyz="0.285 0.45 0.23" rpy="0 0 0"/>
+      <geometry>
+        <box size="0.033 0.033 0.47"/>
+      </geometry>
+      <material name="brown"/>
+    </visual>
+    <collision>
+      <origin xyz="0.285 0.45 0.23" rpy="0 0 0"/>
+      <geometry>
+        <box size="0.033 0.033 0.47"/>
+      </geometry>
+    </collision>
+    <visual>
+      <origin xyz="-0.285 0.45 0.23" rpy="0 0 0"/>
+      <geometry>
+        <box size="0.033 0.033 0.47"/>
+      </geometry>
+      <material name="brown"/>
+    </visual>
+    <collision>
+      <origin xyz="-0.285 0.45 0.23" rpy="0 0 0"/>
+      <geometry>
+        <box size="0.033 0.033 0.47"/>
+      </geometry>
+    </collision>
+    <visual>
+      <origin xyz="0.285 -0.45 0.23" rpy="0 0 0"/>
+      <geometry>
+        <box size="0.033 0.033 0.47"/>
+      </geometry>
+      <material name="brown"/>
+    </visual>
+    <collision>
+      <origin xyz="0.285 -0.45 0.23" rpy="0 0 0"/>
+      <geometry>
+        <box size="0.033 0.033 0.47"/>
+      </geometry>
+    </collision>
+    <visual>
+      <origin xyz="-0.285 -0.45 0.23" rpy="0 0 0"/>
+      <geometry>
+        <box size="0.033 0.033 0.47"/>
+      </geometry>
+      <material name="brown"/>
+    </visual>
+    <collision>
+      <origin xyz="-0.285 -0.45 0.23" rpy="0 0 0"/>
+      <geometry>
+        <box size="0.033 0.033 0.47"/>
+      </geometry>
+    </collision>
+  </link>
+  <joint name="table_to_base" type="fixed">
+    <parent link="bot_base_link"/>  <!-- Hier geändert von base_link zu bot_base_link -->
+    <child link="table_link"/>
+    <origin xyz="0.8 0 0" rpy="0 0 0"/> <!-- 0.8m vor dem Roboter, auf Bodenhöhe -->
+  </joint>
 </robot>

File: ur_simulation_gz/urdf/ur_gz.ros2_control.xacro (robot description, xacro)
@@ -7,5 +7,5 @@
     sim_ignition:=false
     headless_mode:=false
-    initial_positions:=${dict(shoulder_pan_joint=0.0,shoulder_lift_joint=-1.57,elbow_joint=0.0,wrist_1_joint=-1.57,wrist_2_joint=0.0,wrist_3_joint=0.0)}
+    initial_positions:=${xacro.load_yaml(initial_positions_file)}
     use_tool_communication:=false
     script_filename output_recipe_filename

Commit message: added camera, table and tower to sim

File: ur_simulation_gz/urdf/ur5_gripper.urdf.xacro (robot description, xacro)
@@ -39,5 +39,5 @@
    <xacro:arg name="tool_device_name" default="/tmp/ttyUR" />
    <xacro:arg name="tool_tcp_port" default="54321" />
-     <!-- Simulation parameters -->
+   <!-- Simulation parameters -->
    <xacro:arg name="use_fake_hardware" default="false" />
    <xacro:arg name="fake_sensor_commands" default="false" />
@@ -69,10 +69,10 @@
          </material>
        </visual>
-       <!--<collision>
+       <collision>
          <origin rpy="0 0 0" xyz="0 0 0"/>
          <geometry>
            <box size="5 5 0"/>
          </geometry>
-       </collision>-->
+       </collision>
      </link>
      <joint name="ground_plane_joint" type="fixed">
@@ -161,10 +161,10 @@
       </material>
     </visual>
-    <!--<collision>
+    <collision>
       <origin xyz="0 0 0.05" rpy="0 0 0"/>
       <geometry>
         <cylinder length="0.1" radius="0.2"/>
       </geometry>
-    </collision>-->
+    </collision>
   </link>
   <joint name="robot_to_turtlebot_base" type="fixed">
@@ -178,5 +178,5 @@
       <origin xyz="0 0 0.2" rpy="0 0 0"/>
       <geometry>
-        <box size="0.04 0.1 1.2"/>
+        <box size="0.04 0.1 1.0"/>
       </geometry>
       <material name="gray">
@@ -184,15 +184,15 @@
       </material>
     </visual>
-    <!--<collision>
+    <collision>
       <origin xyz="0 0 0.2" rpy="0 0 0"/>
       <geometry>
-        <box size="0.04 0.1 1.2"/>
-      </geometry>
-    </collision> -->
+        <box size="0.04 0.1 1.0"/>
+      </geometry>
+    </collision>
   </link>
   <joint name="pole_to_base" type="fixed">
     <parent link="bot_base_link"/>
     <child link="tower_link"/>
-    <origin xyz="-0.12 0 0.5" rpy="0 0 0"/>
+    <origin xyz="-0.12 0 0.4" rpy="0 0 0"/>
   </joint>
   <!-- Camera -->
@@ -201,5 +201,5 @@
       <origin xyz="0 0 0" rpy="0 0 0"/>
       <geometry>
-        <box size="0.06 0.03 0.02"/>
+        <box size="0.04 0.07 0.02"/>
       </geometry>
       <material name="dark_gray">
@@ -207,15 +207,15 @@
       </material>
     </visual>
-    <!--<collision>
+    <collision>
       <origin xyz="0 0 0" rpy="0 0 0"/>
       <geometry>
         <box size="0.06 0.03 0.02"/>
       </geometry>
-    </collision>-->
+    </collision>
   </link>
   <joint name="camera_on_pole" type="fixed">
     <parent link="tower_link"/>
     <child link="camera_link"/>
-    <origin xyz="0.04 0 0.7" rpy="0 0 0"/>
+    <origin xyz="0.04 0 0.5" rpy="0 0 0"/>
   </joint>
   <!-- Table -->
@@ -292,7 +292,7 @@
   </link>
   <joint name="table_to_base" type="fixed">
-    <parent link="bot_base_link"/>  <!-- Hier geändert von base_link zu bot_base_link -->
+    <parent link="bot_base_link"/>
     <child link="table_link"/>
-    <origin xyz="0.8 0 0" rpy="0 0 0"/> <!-- 0.8m vor dem Roboter, auf Bodenhöhe -->
+    <origin xyz="0.8 0 0" rpy="0 0 0"/>
   </joint>
 </robot>

File: ur_simulation_gz/urdf/ur5_macro.xacro (robot description, xacro)
@@ -54,5 +54,5 @@
     <xacro:if value="${generate_ros2_control_tag}">
       <!-- ros2 control include -->
-      <xacro:include filename="$(find ur_simulation_gz)/urdf/ur_gz.ros2_control.xacro" />
+      <xacro:include filename="$(find ur_simulation_gz)/urdf/ur5_ros2_control.xacro" />
       <!-- ros2 control instance -->
       <xacro:ur_ros2_control
