Commit message: msg type for orchestrator message to MoveItNode

File: ur_simulation_gz/urdf/ur_gz.ros2_control.xacro (robot description, xacro)
@@ -1,298 +1,23 @@
 <?xml version="1.0"?>
-<robot xmlns:xacro="http://wiki.ros.org/xacro" name="ur">
-   <!-- robot name parameter -->
-   <xacro:arg name="name" default="ur"/>
-   <!-- import main macro -->
-   <xacro:include filename="$(find ur_simulation_gz)/urdf/ur5_macro.xacro"/>
-   <!-- possible 'ur_type' values: ur3, ur3e, ur5, ur5e, ur7e, ur10, ur10e, ur12e, ur16e, ur15, ur20, ur30 -->
-   <!-- the default value should raise an error in case this was called without defining the type -->
-   <xacro:arg name="ur_type" default="ur5"/>
-   <!-- parameters -->
-   <xacro:arg name="tf_prefix" default="" />
-   <xacro:arg name="joint_limit_params" default="$(find ur_description)/config/$(arg ur_type)/joint_limits.yaml"/>
-   <xacro:arg name="kinematics_params" default="$(find ur_description)/config/$(arg ur_type)/default_kinematics.yaml"/>
-   <xacro:arg name="physical_params" default="$(find ur_description)/config/$(arg ur_type)/physical_parameters.yaml"/>
-   <xacro:arg name="visual_params" default="$(find ur_description)/config/$(arg ur_type)/visual_parameters.yaml"/>
-   <xacro:arg name="transmission_hw_interface" default=""/>
-   <xacro:arg name="safety_limits" default="false"/>
-   <xacro:arg name="safety_pos_margin" default="0.15"/>
-   <xacro:arg name="safety_k_position" default="20"/>
-   <!-- ros2_control related parameters -->
-   <xacro:arg name="headless_mode" default="false" />
-   <xacro:arg name="robot_ip" default="0.0.0.0" />
-   <xacro:arg name="script_filename" default=""/>
-   <xacro:arg name="output_recipe_filename" default=""/>
-   <xacro:arg name="input_recipe_filename" default=""/>
-   <xacro:arg name="reverse_ip" default="0.0.0.0"/>
-   <xacro:arg name="script_command_port" default="50004"/>
-   <xacro:arg name="reverse_port" default="50001"/>
-   <xacro:arg name="script_sender_port" default="50002"/>
-   <xacro:arg name="trajectory_port" default="50003"/>
-   <!--   tool communication related parameters-->
-   <xacro:arg name="use_tool_communication" default="false" />
-   <xacro:arg name="tool_voltage" default="0" />
-   <xacro:arg name="tool_parity" default="0" />
-   <xacro:arg name="tool_baud_rate" default="115200" />
-   <xacro:arg name="tool_stop_bits" default="1" />
-   <xacro:arg name="tool_rx_idle_chars" default="1.5" />
-   <xacro:arg name="tool_tx_idle_chars" default="3.5" />
-   <xacro:arg name="tool_device_name" default="/tmp/ttyUR" />
-   <xacro:arg name="tool_tcp_port" default="54321" />
-     <!-- Simulation parameters -->
-   <xacro:arg name="use_fake_hardware" default="false" />
-   <xacro:arg name="fake_sensor_commands" default="false" />
-   <xacro:arg name="sim_gazebo" default="true" />
-   <xacro:arg name="sim_ignition" default="false" />
-   <xacro:arg name="simulation_controllers" default="$(find ur_simulation_gz)/config/ur5_controllers_gripper.yaml" />
-   <!-- initial position for simulations (Fake Hardware, Gazebo, Ignition) -->
-   <xacro:arg name="initial_positions_file" default="$(find ur_simulation_gz)/config/initial_positions.yaml"/>
-   <!-- convert to property to use substitution in function -->
-   <xacro:property name="initial_positions_file" default="$(arg initial_positions_file)"/>
-   <xacro:property name="is_sim_gazebo" value="$(arg sim_gazebo)"/>
-   <xacro:property name="is_sim_ignition" value="$(arg sim_ignition)"/>
-   <!-- create link fixed to the "world" -->
-   <link name="world" />
-   <joint name="world_to_bot_base" type="fixed">
-    <parent link="world"/>
-    <child link="bot_base_link"/>
-    <origin xyz="0 0 0" rpy="0 0 0"/>
-  </joint>
-   <xacro:if value="${is_sim_gazebo or is_sim_ignition}">
-     <link name="ground_plane">
-       <visual>
-         <origin rpy="0 0 0" xyz="0 0 0"/>
-         <geometry>
-           <box size="5 5 0"/>
-         </geometry>
-         <material name="ground_white">
-           <color rgba="1 1 1 0.5"/>
-         </material>
-       </visual>
-       <collision>
-         <origin rpy="0 0 0" xyz="0 0 0"/>
-         <geometry>
-           <box size="5 5 0"/>
-         </geometry>
-       </collision>
-     </link>
-     <joint name="ground_plane_joint" type="fixed">
-       <origin xyz="0 0 -0.01" rpy="0 0 0"/>
-       <parent link="world"/>
-       <child link="ground_plane"/>
-     </joint>
-   </xacro:if>
-   <!-- arm -->
-   <xacro:ur_robot
-     name="$(arg name)"
-     tf_prefix="$(arg tf_prefix)"
-     parent="world"
-     joint_limits_parameters_file="$(arg joint_limit_params)"
-     kinematics_parameters_file="$(arg kinematics_params)"
-     physical_parameters_file="$(arg physical_params)"
-     visual_parameters_file="$(arg visual_params)"
-     transmission_hw_interface="$(arg transmission_hw_interface)"
-     safety_limits="$(arg safety_limits)"
-     safety_pos_margin="$(arg safety_pos_margin)"
-     safety_k_position="$(arg safety_k_position)"
-     use_fake_hardware="$(arg use_fake_hardware)"
-     fake_sensor_commands="$(arg fake_sensor_commands)"
-     sim_gazebo="$(arg sim_gazebo)"
-     sim_ignition="$(arg sim_ignition)"
-     headless_mode="$(arg headless_mode)"
-     initial_positions="${xacro.load_yaml(initial_positions_file)}"
-     use_tool_communication="$(arg use_tool_communication)"
-     tool_voltage="$(arg tool_voltage)"
-     tool_parity="$(arg tool_parity)"
-     tool_baud_rate="$(arg tool_baud_rate)"
-     tool_stop_bits="$(arg tool_stop_bits)"
-     tool_rx_idle_chars="$(arg tool_rx_idle_chars)"
-     tool_tx_idle_chars="$(arg tool_tx_idle_chars)"
-     tool_device_name="$(arg tool_device_name)"
-     tool_tcp_port="$(arg tool_tcp_port)"
-     robot_ip="$(arg robot_ip)"
-     script_filename="$(arg script_filename)"
-     output_recipe_filename="$(arg output_recipe_filename)"
-     input_recipe_filename="$(arg input_recipe_filename)"
-     reverse_ip="$(arg reverse_ip)"
-     script_command_port="$(arg script_command_port)"
-     reverse_port="$(arg reverse_port)"
-     script_sender_port="$(arg script_sender_port)"
-     trajectory_port="$(arg trajectory_port)"
-     >
-     <origin xyz="0 0 0" rpy="0 0 0" />         <!-- position robot in the world -->
-   </xacro:ur_robot>
-   <xacro:if value="$(arg sim_gazebo)">
-    <!-- Gazebo plugins -->
-    <gazebo reference="world">
-    </gazebo>
-    <gazebo>
-      <plugin filename="libgazebo_ros2_control.so" name="gazebo_ros2_control">
-        <parameters>$(arg simulation_controllers)</parameters>
-      </plugin>
-    </gazebo>
-  </xacro:if>
-  <xacro:if value="$(arg sim_ignition)">
-    <!-- Gazebo plugins -->
-    <gazebo reference="world">
-    </gazebo>
-    <gazebo>
-      <plugin filename="libign_ros2_control-system.so" name="ign_ros2_control::IgnitionROS2ControlPlugin">
-        <parameters>$(arg simulation_controllers)</parameters>
-        <controller_manager_node_name>$(arg tf_prefix)controller_manager</controller_manager_node_name>
-      </plugin>
-    </gazebo>
-  </xacro:if>
-  <xacro:arg name="use_fake_hardware" default="true" />
-  <xacro:arg name="com_port" default="/dev/ttyUSB0" />
-  <!-- Import macros -->
-  <xacro:include filename="$(find ur_simulation_gz)/urdf/robotiq_gripper_macro.xacro" />
-  <xacro:robotiq_gripper name="RobotiqGripperHardwareInterface" prefix="" parent="tool0" use_fake_hardware="$(arg use_fake_hardware)" com_port="$(arg com_port)" sim_gazebo="$(arg sim_gazebo)">
-    <origin xyz="0 0 0" rpy="0 0 0" />
-  </xacro:robotiq_gripper>
-  <!-- Base -->
-  <link name="bot_base_link">
-    <visual>
-      <origin xyz="0 0 0.05" rpy="0 0 0"/>
-      <geometry>
-        <cylinder length="0.1" radius="0.2"/>
-      </geometry>
-      <material name="dark_gray">
-        <color rgba="0.2 0.2 0.2 1"/>
-      </material>
-    </visual>
-    <!--<collision>
-      <origin xyz="0 0 0.05" rpy="0 0 0"/>
-      <geometry>
-        <cylinder length="0.1" radius="0.2"/>
-      </geometry>
-    </collision>-->
-  </link>
-  <joint name="robot_to_turtlebot_base" type="fixed">
-    <parent link="bot_base_link"/>
-    <child link="base_link"/>  <!-- Ur5 Base -->
-    <origin xyz="0 0 0.1" rpy="0 0 0"/>
-  </joint>
-  <!-- Tower -->
-  <link name="tower_link">
-    <visual>
-      <origin xyz="0 0 0.2" rpy="0 0 0"/>
-      <geometry>
-        <box size="0.04 0.1 1.2"/>
-      </geometry>
-      <material name="gray">
-        <color rgba="0.5 0.5 0.5 1"/>
-      </material>
-    </visual>
-    <!--<collision>
-      <origin xyz="0 0 0.2" rpy="0 0 0"/>
-      <geometry>
-        <box size="0.04 0.1 1.2"/>
-      </geometry>
-    </collision> -->
-  </link>
-  <joint name="pole_to_base" type="fixed">
-    <parent link="bot_base_link"/>
-    <child link="tower_link"/>
-    <origin xyz="-0.12 0 0.5" rpy="0 0 0"/>
-  </joint>
-  <!-- Camera -->
-  <link name="camera_link">
-    <visual>
-      <origin xyz="0 0 0" rpy="0 0 0"/>
-      <geometry>
-        <box size="0.06 0.03 0.02"/>
-      </geometry>
-      <material name="dark_gray">
-        <color rgba="0.2 0.2 0.2 1"/>
-      </material>
-    </visual>
-    <!--<collision>
-      <origin xyz="0 0 0" rpy="0 0 0"/>
-      <geometry>
-        <box size="0.06 0.03 0.02"/>
-      </geometry>
-    </collision>-->
-  </link>
-  <joint name="camera_on_pole" type="fixed">
-    <parent link="tower_link"/>
-    <child link="camera_link"/>
-    <origin xyz="0.04 0 0.7" rpy="0 0 0"/>
-  </joint>
-  <!-- Table -->
-    <link name="table_link">
-    <!-- Tischplatte -->
-    <visual>
-      <origin xyz="0 0 0.47" rpy="0 0 0"/>
-      <geometry>
-        <box size="0.67 1.0 0.033"/>
-      </geometry>
-      <material name="brown">
-        <color rgba="0.55 0.27 0.07 1"/>
-      </material>
-    </visual>
-    <collision>
-      <origin xyz="0 0 0.47" rpy="0 0 0"/>
-      <geometry>
-        <box size="0.67 1.0 0.033"/>
-      </geometry>
-    </collision>
-    <!-- Tischbeine -->
-    <visual>
-      <origin xyz="0.285 0.45 0.23" rpy="0 0 0"/>
-      <geometry>
-        <box size="0.033 0.033 0.47"/>
-      </geometry>
-      <material name="brown"/>
-    </visual>
-    <collision>
-      <origin xyz="0.285 0.45 0.23" rpy="0 0 0"/>
-      <geometry>
-        <box size="0.033 0.033 0.47"/>
-      </geometry>
-    </collision>
-    <visual>
-      <origin xyz="-0.285 0.45 0.23" rpy="0 0 0"/>
-      <geometry>
-        <box size="0.033 0.033 0.47"/>
-      </geometry>
-      <material name="brown"/>
-    </visual>
-    <collision>
-      <origin xyz="-0.285 0.45 0.23" rpy="0 0 0"/>
-      <geometry>
-        <box size="0.033 0.033 0.47"/>
-      </geometry>
-    </collision>
-    <visual>
-      <origin xyz="0.285 -0.45 0.23" rpy="0 0 0"/>
-      <geometry>
-        <box size="0.033 0.033 0.47"/>
-      </geometry>
-      <material name="brown"/>
-    </visual>
-    <collision>
-      <origin xyz="0.285 -0.45 0.23" rpy="0 0 0"/>
-      <geometry>
-        <box size="0.033 0.033 0.47"/>
-      </geometry>
-    </collision>
-    <visual>
-      <origin xyz="-0.285 -0.45 0.23" rpy="0 0 0"/>
-      <geometry>
-        <box size="0.033 0.033 0.47"/>
-      </geometry>
-      <material name="brown"/>
-    </visual>
-    <collision>
-      <origin xyz="-0.285 -0.45 0.23" rpy="0 0 0"/>
-      <geometry>
-        <box size="0.033 0.033 0.47"/>
-      </geometry>
-    </collision>
-  </link>
-  <joint name="table_to_base" type="fixed">
-    <parent link="bot_base_link"/>  <!-- Hier geändert von base_link zu bot_base_link -->
-    <child link="table_link"/>
-    <origin xyz="0.8 0 0" rpy="0 0 0"/> <!-- 0.8m vor dem Roboter, auf Bodenhöhe -->
-  </joint>
+<robot xmlns:xacro="http://www.ros.org/wiki/xacro">
+  <xacro:include filename="$(find ur_description)/urdf/inc/ur_joint_control.xacro" />
+  <xacro:macro name="ur_ros2_control" params="
+    name
+    tf_prefix
+    transmission_hw_interface:=hardware_interface/PositionJointInterface
+    initial_positions:=${dict(shoulder_pan_joint=0.0,shoulder_lift_joint=-1.57,elbow_joint=0.0,wrist_1_joint=-1.57,wrist_2_joint=0.0,wrist_3_joint=0.0)}
+    ">
+    <!-- Add URDF transmission elements (for ros_control) -->
+    <!--<xacro:ur_arm_transmission prefix="${prefix}" hw_interface="${transmission_hw_interface}" />-->
+    <!-- Placeholder for ros2_control transmission which don't yet exist -->
+    <ros2_control name="${name}" type="system">
+      <hardware>
+        <plugin>gz_ros2_control/GazeboSimSystem</plugin>
+      </hardware>
+      <xacro:ur_joint_control_description
+        tf_prefix="${tf_prefix}"
+        initial_positions="${initial_positions}"
+      />
+      </ros2_control>
+  </xacro:macro>
 </robot>

File: ur_simulation_gz/urdf/ur_gz.urdf.xacro (robot description, xacro)
@@ -21,4 +21,7 @@
   <xacro:arg name="simulation_controllers" default="" />
   <xacro:arg name="ros_namespace" default="" />
+  <xacro:arg name="use_fake_hardware" default="false"/>
+  <xacro:arg name="com_port" default="/dev/ttyUSB0"/>
+  <xacro:arg name="sim_gazebo" default="true"/>
   <!-- create link fixed to the "world" -->
   <link name="world" />
@@ -45,9 +48,32 @@
     <child link="ground_plane"/>
   </joint>
+  <!-- Base -->
+  <link name="bot_link">
+    <visual>
+      <origin xyz="0 0 0.05" rpy="0 0 0"/>
+      <geometry>
+        <cylinder length="0.1" radius="0.2"/>
+      </geometry>
+      <material name="dark_gray">
+        <color rgba="0.2 0.2 0.2 1"/>
+      </material>
+    </visual>
+    <collision>
+      <origin xyz="0 0 0.05" rpy="0 0 0"/>
+      <geometry>
+        <cylinder length="0.1" radius="0.2"/>
+      </geometry>
+    </collision>
+  </link>
+  <joint name="world_to_base" type="fixed">
+    <parent link="ground_plane"/>
+    <child link="bot_link"/>
+    <origin xyz="0 0 0" rpy="0 0 0"/>
+  </joint>
   <!-- arm -->
   <xacro:ur_robot
     name="$(arg name)"
     tf_prefix="$(arg tf_prefix)"
-    parent="world"
+    parent="bot_link"
     joint_limits_parameters_file="$(arg joint_limit_params)"
     kinematics_parameters_file="$(arg kinematics_params)"
@@ -77,3 +103,131 @@
     transmission_hw_interface="$(arg transmission_hw_interface)"
   />
+  <!-- Import macros -->
+  <xacro:include filename="$(find ur_simulation_gz)/urdf/robotiq_gripper_macro.xacro" />
+  <xacro:robotiq_gripper name="RobotiqGripperHardwareInterface" prefix="" parent="tool0" use_fake_hardware="$(arg use_fake_hardware)" com_port="$(arg com_port)" sim_gazebo="$(arg sim_gazebo)">
+    <origin xyz="0 0 0" rpy="0 0 0" />
+  </xacro:robotiq_gripper>
+  <!-- Tower -->
+  <link name="tower_link">
+    <visual>
+      <origin xyz="0 0 0.2" rpy="0 0 0"/>
+      <geometry>
+        <box size="0.04 0.1 1.0"/>
+      </geometry>
+      <material name="gray">
+        <color rgba="0.5 0.5 0.5 1"/>
+      </material>
+    </visual>
+    <collision>
+      <origin xyz="0 0 0.2" rpy="0 0 0"/>
+      <geometry>
+        <box size="0.04 0.1 1.0"/>
+      </geometry>
+    </collision>
+  </link>
+  <joint name="pole_to_base" type="fixed">
+    <parent link="bot_link"/>
+    <child link="tower_link"/>
+    <origin xyz="-0.12 0 0.4" rpy="0 0 0"/>
+  </joint>
+  <!-- Camera -->
+  <link name="camera_link">
+    <visual>
+      <origin xyz="0 0 0" rpy="0 0 0"/>
+      <geometry>
+        <box size="0.04 0.07 0.02"/>
+      </geometry>
+      <material name="dark_gray">
+        <color rgba="0.2 0.2 0.2 1"/>
+      </material>
+    </visual>
+    <collision>
+      <origin xyz="0 0 0" rpy="0 0 0"/>
+      <geometry>
+        <box size="0.06 0.03 0.02"/>
+      </geometry>
+    </collision>
+  </link>
+  <joint name="camera_on_pole" type="fixed">
+    <parent link="tower_link"/>
+    <child link="camera_link"/>
+    <origin xyz="0.04 0 0.5" rpy="0 0 0"/>
+  </joint>
+  <!-- Table -->
+    <link name="table_link">
+    <!-- Tischplatte -->
+    <visual>
+      <origin xyz="0 0 0.47" rpy="0 0 0"/>
+      <geometry>
+        <box size="0.67 1.0 0.033"/>
+      </geometry>
+      <material name="brown">
+        <color rgba="0.55 0.27 0.07 1"/>
+      </material>
+    </visual>
+    <collision>
+      <origin xyz="0 0 0.47" rpy="0 0 0"/>
+      <geometry>
+        <box size="0.67 1.0 0.033"/>
+      </geometry>
+    </collision>
+    <!-- Tischbeine -->
+    <visual>
+      <origin xyz="0.285 0.45 0.23" rpy="0 0 0"/>
+      <geometry>
+        <box size="0.033 0.033 0.47"/>
+      </geometry>
+      <material name="brown"/>
+    </visual>
+    <collision>
+      <origin xyz="0.285 0.45 0.23" rpy="0 0 0"/>
+      <geometry>
+        <box size="0.033 0.033 0.47"/>
+      </geometry>
+    </collision>
+    <visual>
+      <origin xyz="-0.285 0.45 0.23" rpy="0 0 0"/>
+      <geometry>
+        <box size="0.033 0.033 0.47"/>
+      </geometry>
+      <material name="brown"/>
+    </visual>
+    <collision>
+      <origin xyz="-0.285 0.45 0.23" rpy="0 0 0"/>
+      <geometry>
+        <box size="0.033 0.033 0.47"/>
+      </geometry>
+    </collision>
+    <visual>
+      <origin xyz="0.285 -0.45 0.23" rpy="0 0 0"/>
+      <geometry>
+        <box size="0.033 0.033 0.47"/>
+      </geometry>
+      <material name="brown"/>
+    </visual>
+    <collision>
+      <origin xyz="0.285 -0.45 0.23" rpy="0 0 0"/>
+      <geometry>
+        <box size="0.033 0.033 0.47"/>
+      </geometry>
+    </collision>
+    <visual>
+      <origin xyz="-0.285 -0.45 0.23" rpy="0 0 0"/>
+      <geometry>
+        <box size="0.033 0.033 0.47"/>
+      </geometry>
+      <material name="brown"/>
+    </visual>
+    <collision>
+      <origin xyz="-0.285 -0.45 0.23" rpy="0 0 0"/>
+      <geometry>
+        <box size="0.033 0.033 0.47"/>
+      </geometry>
+    </collision>
+  </link>
+  <joint name="table_to_base" type="fixed">
+    <parent link="ground_plane"/>
+    <child link="table_link"/>
+    <origin xyz="0.8 0 0" rpy="0 0 0"/>
+  </joint>
 </robot>
